File: PUSH BUTTONS.kicad_sch (KiCad schematic)
At the start: 136 parts, among them SW1 RotaryEncoder_Switch, SW2 RotaryEncoder_Switch, SW3 RotaryEncoder_Switch, SW4 RotaryEncoder_Switch, SW5 RotaryEncoder_Switch, U1 IS31FL3733-QF, U2 IS31FL3733-QF

Commit message: schmtcs vsn1
Parts:
- removed C19: 47uF, PCM_JLCPCB:C_0805, symbol PCM_JLCPCB-Capacitors:0805,47uF
- removed C3: 100nF, PCM_JLCPCB:C_0402, symbol PCM_JLCPCB-Capacitors:0402,100nF
- C1: value 47uF -> 100n 16V; footprint PCM_JLCPCB:C_0805 -> moshte:C_0603
- C17, C18, C21, C22, C25, C26, C4: value 100nF -> 100n 16V; footprint PCM_JLCPCB:C_0402 -> moshte:C_0402
- C2, C20, C23, C24, C5, C6: value 470nF -> 470n 10V; footprint PCM_JLCPCB:C_0402 -> moshte:C_0402
- R1, R10, R11, R12, R13, R14, R15, R2, R8, R9: footprint PCM_JLCPCB:R_0402 -> moshte:R_0402
- R16, R17: footprint PCM_JLCPCB:R_0603 -> moshte:R_0603
Connections:
- net +3.3V: now also C18.2, C26.2, R1.2, R2.2, U1.39 (VIO), U2.39 (VIO)
- net +VSW: no longer C18.1, C26.1, R1.1, R2.1, U1.39 (VIO), U2.39 (VIO)
- net GND: now also C18.1, C26.1; no longer C18.2, C26.2
- net LEDS_SHUTDOWN: now also R1.1, R2.1; no longer R1.2, R2.2
- net SCL renamed DRV1_SCL
- net DRV1_SCL: no longer R12.2, U2.42 (SCL)
- net SDA renamed DRV1_SDA
- net DRV1_SDA: no longer R13.2, U2.41 (SDA)
- new net DRV2_SCL: R12.2, U2.42 (SCL)
- new net DRV2_SDA: R13.2, U2.41 (SDA)
Other:
- moved on the sheet: C1, C17, C18, C2, C20, C21, C22, C23, C24, C25, C26, C4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
