File: Chord Board Controller.kicad_pcb (KiCad board)
At the start: 4 copper layers, 207 x 149.9 mm, 197 parts, among them J4 HRO_TYPE-C-31-M-14, J6 TC2030_SWD, J8 Battery, Q13 2N7002, SW1 RotaryEncoder_Switch, SW2 RotaryEncoder_Switch, SW3 RotaryEncoder_Switch, SW4 RotaryEncoder_Switch, SW5 RotaryEncoder_Switch, SW6 SW_SPST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

Commit message: schmtcs vsn1
Parts:
- added C10: 22u, moshte:C_0603, F.Cu at (291.6, 127.0)
- added C11: 22u, moshte:C_0603, F.Cu at (291.6, 129.5)
- added C12: 22u, moshte:C_0603, F.Cu at (291.6, 132.0)
- added C28: 100n 16V, moshte:C_0603, F.Cu at (291.6, 134.5)
- added C29: 100n 16V, moshte:R_0603, F.Cu at (291.6, 137.0)
- added C30: 4u7 25V, moshte:C_0603, F.Cu at (291.6, 139.5)
- added C31: 4u7, moshte:C_0603, F.Cu at (295.6, 127.0)
- added C32: 100n 16V, moshte:C_0402, F.Cu at (309.0, 142.5)
- added C33: 4u7, moshte:C_0603, F.Cu at (295.6, 129.5)
- added C34: 22u, moshte:C_0603, F.Cu at (295.6, 132.0)
- added D3: SS110, moshte:DIOM4325X250N, F.Cu at (294.2, 142.8)
- added FB1: 120R, moshte:FB_0603, F.Cu at (295.6, 134.5)
- added J1: 5 Pin Header 2.54mm, moshte:5 Pin Header 2.54mm, F.Cu at (296.7, 123.7)
- added L1: 470n, moshte:L_0402, F.Cu at (309.0, 130.6)
- added L2: 470n, moshte:L_0402, F.Cu at (309.0, 132.6)
- added PG_LED1: Blue, LED_THT:LED_D1.8mm_W1.8mm_H2.4mm_Horizontal_O6.35mm_Z8.2mm, F.Cu at (303.3, 131.3)
- added R21: 10k, moshte:R_0402, F.Cu at (309.0, 134.6)
- added R22: 10k, moshte:R_0402, F.Cu at (309.0, 136.5)
- added R23: 10kΩ, moshte:R_0402, F.Cu at (309.0, 138.5)
- added R24: 10k, moshte:R_0402, F.Cu at (309.0, 140.5)
- added R25: 1k5, moshte:R_0603, F.Cu at (295.6, 137.0)
- added R26: 511k, moshte:R_0603, F.Cu at (295.6, 139.5)
- added R27: 91k, moshte:R_0603, F.Cu at (299.6, 127.0)
- added R28: 806k, moshte:R_0603, F.Cu at (299.6, 129.5)
- added R29: 91k, moshte:R_0603, F.Cu at (299.6, 132.0)
- added U3: TPS63805YFFR, moshte:BGA15N40P5X3_225X134X62N, F.Cu at (303.6, 127.7)
- added U4: TPS63805YFFR, moshte:BGA15N40P5X3_225X134X62N, F.Cu at (307.1, 127.7)
- C1: value 47uF -> 100n 16V; footprint PCM_JLCPCB:C_0805 -> moshte:C_0603
- C13, C15: value 4u7 -> 4u7 25V; footprint Capacitor_SMD:C_0603_1608Metric -> moshte:C_0603
- C14: footprint Capacitor_SMD:C_0603_1608Metric -> moshte:C_0603
- C16: value 4.7uF -> 4.7u 10V; footprint PCM_JLCPCB:C_0402 -> moshte:C_0402
- C17, C18, C21, C22, C25, C26, C4, C8, C9: value 100nF -> 100n 16V; footprint PCM_JLCPCB:C_0402 -> moshte:C_0402
- C2, C20, C23, C24, C5, C6: value 470nF -> 470n 10V; footprint PCM_JLCPCB:C_0402 -> moshte:C_0402
- C27: value 100n -> 100n 16V; footprint Capacitor_SMD:C_0402_1005Metric_Pad0.74x0.62mm_HandSolder -> moshte:C_0402
- C7: value 10uF -> 10u 6v3; footprint PCM_JLCPCB:C_0402 -> moshte:C_0402
- CHG_LED1: renamed from LED_CHG1; value Orange -> Red
- J4: footprint PCM_marbastlib-various:USB_C_Receptacle_HRO_TYPE-C-31-M-14 -> marbastlib-various:USB_C_Receptacle_HRO_TYPE-C-31-M-14
- J8: value Battery -> Batt_1S
- R1, R10, R11, R12, R13, R14, R15, R2, R8, R9: footprint PCM_JLCPCB:R_0402 -> moshte:R_0402
- R16, R17, R35: footprint PCM_JLCPCB:R_0603 -> moshte:R_0603
- R18: footprint Resistor_SMD:R_0402_1005Metric_Pad0.72x0.64mm_HandSolder -> moshte:R_0402
- R19, R3, R32, R33, R34, R4, R40, R5, R6, R7: footprint Resistor_SMD:R_0402_1005Metric -> moshte:R_0402
- R20: footprint PCM_JLCPCB:R_0402 -> moshte:R_0402; moved to B.Cu
- R39: value 806k -> 1.6M; footprint Resistor_SMD:R_0402_1005Metric -> moshte:R_0402
- R44, R48, R49, R50: footprint Resistor_SMD:R_0603_1608Metric_Pad0.98x0.95mm_HandSolder -> moshte:R_0603
- R46: value 1k5 -> 1k1 1%; footprint Resistor_SMD:R_0603_1608Metric_Pad0.98x0.95mm_HandSolder -> moshte:R_0603
- R47: value 3k9 -> 1k5 1%; footprint Resistor_SMD:R_0603_1608Metric_Pad0.98x0.95mm_HandSolder -> moshte:R_0603
- moved R20 17.0 mm to (78.0, 148.6), turned to -90 degrees
Connections:
- C13 pad 1: +5V -> +VUSB
- C18 pad 1: +VSW -> GND
- C18 pad 2: GND -> +3.3V
- C26 pad 1: +VSW -> GND
- C26 pad 2: GND -> +3.3V
- CHG_LED1 pad 1: +BATT -> Net-(CHG_LED1-K)
- J4 pad A4: VBUS -> +VBUS
- J4 pad A9: VBUS -> +VBUS
- J4 pad B4: VBUS -> +VBUS
- J4 pad B9: VBUS -> +VBUS
- R1 pad 1: +VSW -> LEDS_SHUTDOWN
- R1 pad 2: LEDS_SHUTDOWN -> +3.3V
- R12 pad 1: +VSW -> +3.3V
- R13 pad 1: +VSW -> +3.3V
- R16 pad 1: +VSW -> +3.3V
- R17 pad 1: +VSW -> +3.3V
- R2 pad 1: +VSW -> LEDS_SHUTDOWN
- R2 pad 2: LEDS_SHUTDOWN -> +3.3V
- R32 pad 1: +5V -> + VUSB
- R44 pad 1: +BATT -> Net-(CHG_LED1-K)
- R49 pad 1: +5V -> +VUSB
- R8 pad 1: +VSW -> +3.3V
- R9 pad 1: +VSW -> +3.3V
- U1 pad 39: +VSW -> +3.3V
- U2 pad 39: +VSW -> +3.3V
- U5 pad 3: unconnected-(U5-IO2-Pad3) -> +VBUS
- U8 pad 13: +5V -> +VUSB
- U8 pad 14: Net-(U8-TMR) -> unconnected-(U8-TMR-Pad14)
- U8 pad 4: GND -> Net-(U8-~{CE})
- U8 pad 5: GND -> Net-(U8-EN2)
- U8 pad 6: +VSW -> Net-(U8-EN1)
- U8 pad 7: unconnected-(U8-~{PGOOD}-Pad7) -> Net-(U8-~{PGOOD})
Routing:
- net Blue4: track 199.4 -> 243.7 mm, vias 11 -> 13
- net Green5: track 237.4 -> 251.9 mm, vias 15 -> 17
- net Red3: track 200.5 -> 212.9 mm, vias 12 -> 16
- net CS7_D2: track 138.3 -> 131.4 mm
- net Green4: track 209.2 -> 215.4 mm, vias 14 -> 16
- net Red5: track 234.0 -> 239.1 mm, vias 15 -> 17
- net unconnected-(U8-TMR-Pad14): track 0.00 -> 4.50 mm
- net Net-(U8-TMR): track 4.78 -> 0.27 mm
- net Green3: track 234.6 -> 230.8 mm, vias 14 -> 20
- net RST: track 51.0 -> 54.5 mm
- net CS8_D2: track 111.3 -> 114.2 mm
- net ROW5: track 377.4 -> 379.4 mm, vias 6 -> 8
- net Blue5: track 205.2 -> 206.5 mm, vias 10 -> 14
- net +3.3V: track 62.2 -> 63.3 mm
- net Red4: track 201.6 -> 202.6 mm, vias 12 -> 14
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
Commit message: gnd cutiings rmvd
Parts:
- removed F1: 500mA, Fuse:Fuse_0805_2012Metric
- removed J6: TC2030_SWD, PCM_marbastlib-various:CON_TC2030_outlined
- removed R43: 10k, Resistor_SMD:R_0603_1608Metric_Pad0.98x0.95mm_HandSolder
- removed R45: 47k, Resistor_SMD:R_0603_1608Metric_Pad0.98x0.95mm_HandSolder
- C14, C33: value 4u7 -> 4u7 25V
- C30, R21, R22, R23, R24, R25: moved to B.Cu
- C31: value 4u7 -> 4u7 25V; moved to B.Cu
- PG_LED1: footprint LED_THT:LED_D1.8mm_W1.8mm_H2.4mm_Horizontal_O6.35mm_Z8.2mm -> moshte:LED_0603; moved to B.Cu
- moved SWD 223.4 mm to (75.2, 153.1), turned to 90 degrees
- moved D3 139.2 mm to (186.6, 54.5)
- moved FB1 136.6 mm to (186.4, 52.3)
- moved C28 135.7 mm to (184.1, 51.6), turned to 90 degrees
- moved C29 133.8 mm to (188.6, 51.6), turned to 90 degrees
- moved R21 76.3 mm to (256.3, 79.4), turned to 90 degrees
- moved R24 74.1 mm to (266.0, 80.2)
- moved R23 71.9 mm to (261.6, 84.5), turned to 90 degrees
- moved R22 71.2 mm to (260.4, 84.5), turned to 90 degrees
- moved C30 64.3 mm to (263.5, 81.7)
- moved R25 60.9 mm to (260.8, 87.0)
- moved PG_LED1 60.4 mm to (260.8, 88.4), turned to 180 degrees
- moved C31 59.8 mm to (256.3, 81.8), turned to -90 degrees
- moved R32 49.0 mm to (209.1, 53.1), turned to 180 degrees
- moved LED3 46.5 mm to (204.2, 53.1)
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- renumbered J8 to BATT_1S, J1 to SWD
Connections:
- C29 pad 1: + VUSB -> +VUSB
- FB1 pad 2: + VUSB -> +VUSB
- R12 pad 2: SCL -> DRV2_SCL
- R13 pad 2: SDA -> DRV2_SDA
- R32 pad 1: + VUSB -> +VUSB
- R8 pad 2: SCL -> DRV1_SCL
- R9 pad 2: SDA -> DRV1_SDA
- U1 pad 41: SDA -> DRV1_SDA
- U1 pad 42: SCL -> DRV1_SCL
- U2 pad 41: SDA -> DRV2_SDA
- U2 pad 42: SCL -> DRV2_SCL
- U7 pad 11: unconnected-(U7-P0.31-LF-A-Pad11) -> DRV2_SDA
- U7 pad 12: unconnected-(U7-P0.04-A-Pad12) -> DRV2_SCL
- U7 pad 13: SCL -> DRV1_SCL
- U7 pad 15: SDA -> DRV1_SDA
Routing:
- net +5V: track 306.3 -> 2.79 mm, vias 11 -> 0
- net (no net): track 0.00 -> 302.4 mm, vias 2 -> 12
- net +VSW: track 433.1 -> 144.8 mm, vias 24 -> 5
- net SCL: track 153.6 -> 0.00 mm, vias 7 -> 0
- net SDA: track 148.8 -> 0.00 mm, vias 2 -> 0
- net +BATT: track 148.1 -> 27.7 mm, vias 6 -> 2
- net +VUSB: track 0.00 -> 119.9 mm, vias 0 -> 2
- net Net-(CHG_LED1-K): track 0.00 -> 81.7 mm, vias 0 -> 2
- net GND: track 107.1 -> 42.4 mm, vias 67 -> 380
- net Blue4: track 243.7 -> 273.7 mm, vias 13 -> 20
- net Blue3: track 190.2 -> 208.6 mm, vias 13 -> 20
- net Blue5: track 206.5 -> 216.7 mm
- net VBUS: track 10.2 -> 0.00 mm, vias 2 -> 0
- net Green3: track 230.8 -> 240.8 mm, vias 20 -> 22
- net Red5: track 239.1 -> 248.9 mm
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- added copper zone on F.Cu, net +VBUS
