File: Chord Board Controller.kicad_pcb (KiCad board)
At the start: 4 copper layers, 207 x 149.9 mm, 220 parts, among them J4 HRO_TYPE-C-31-M-14, Q13 2N7002, SW1 RotaryEncoder_Switch, SW2 RotaryEncoder_Switch, SW3 RotaryEncoder_Switch, SW4 RotaryEncoder_Switch, SW5 RotaryEncoder_Switch, SW6 SW_SPST, SW7 RST, SW8 SW_SPDT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

Commit message: power done
Parts:
- removed the C10 at (109.5, 112.5)
- removed the C12 at (102.3, 111.6)
- C10, C11, C12, C34, L1, L2, R26, R27, R28, R29, U3, U4: moved to B.Cu
- moved C32 218.6 mm to (90.6, 134.5), turned to -90 degrees
- moved L2 104.7 mm to (223.2, 72.7)
- moved U4 98.5 mm to (223.2, 76.0), turned to 90 degrees
- moved L1 96.8 mm to (231.5, 72.7)
- moved C34 93.6 mm to (221.7, 74.5)
- moved R28 93.2 mm to (221.7, 78.2)
- moved R29 92.3 mm to (224.5, 78.2)
- moved R26 89.7 mm to (230.1, 78.2)
- moved U3 88.7 mm to (231.4, 76.0), turned to 90 degrees
- moved C12 88.4 mm to (224.5, 74.5), turned to 180 degrees
- moved R27 82.7 mm to (232.8, 78.2)
- moved C11 82.5 mm to (230.1, 74.4)
- moved C10 78.8 mm to (232.8, 74.4), turned to 180 degrees
- moved C33 47.8 mm to (264.3, 93.3), turned to -90 degrees
- moved U5 40.7 mm to (166.8, 54.1), turned to -90 degrees
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- renumbered SWD to J1, BATT_1S to J8
Routing:
- net +5V: track 2.79 -> 88.5 mm, vias 0 -> 4
- net GND: track 42.4 -> 85.5 mm, vias 380 -> 435
- net +VSW: track 144.8 -> 177.4 mm, vias 5 -> 8
- net (no net): track 302.4 -> 279.9 mm, vias 12 -> 9
- net DRV1_SCL: track 0.00 -> 10.4 mm, vias 0 -> 2
- net DRV1_SDA: track 0.00 -> 10.0 mm
- net +VBUS: track 3.33 -> 10.8 mm
- net +3.3V: track 62.1 -> 69.5 mm
- net USB-D+: track 140.1 -> 146.4 mm
- net USB-D-: track 138.9 -> 144.3 mm
- net Net-(L2-Pad1): track 0.00 -> 4.91 mm
- net Net-(L2-Pad2): track 0.00 -> 4.60 mm
- net Net-(L1-Pad2): track 0.00 -> 4.45 mm
- net Net-(L1-Pad1): track 0.00 -> 4.39 mm
- net CS1_D2: track 156.0 -> 159.4 mm
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
Commit message: Routing done
Parts:
- removed the C11 at (103.7, 111.6)
- removed C3: 100nF, PCM_JLCPCB:C_0402
- removed U6: XC6206PxxxMR, Package_TO_SOT_SMD:SOT-23
- moved R8 3.45 mm to (130.2, 111.3)
- moved R9 2.29 mm to (130.2, 112.5)
- moved R10 2.05 mm to (135.4, 115.2), turned to 180 degrees
- moved R2 2.04 mm to (221.8, 111.8), turned to 0 degrees
- moved C6 2.01 mm to (127.5, 119.0)
- moved C17 2.01 mm to (127.5, 120.0)
- moved R14 1.96 mm to (221.8, 113.0), turned to 180 degrees
- moved R12 1.83 mm to (217.0, 109.8)
- moved R13 1.83 mm to (217.0, 110.8)
- moved C1 1.64 mm to (132.8, 124.6)
- moved C4 1.46 mm to (128.9, 114.7)
- moved C5 1.46 mm to (128.0, 114.7)
- moved R1 1.40 mm to (134.3, 113.7), turned to 90 degrees
- moved C18 1.10 mm to (130.7, 114.7), turned to -90 degrees
- moved R17 0.74 mm to (221.5, 108.0)
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Routing:
- net +VSW: track 177.4 -> 624.9 mm, vias 8 -> 18
- net (no net): track 279.9 -> 0.00 mm, vias 9 -> 0
- net +3.3V: track 69.5 -> 246.9 mm, vias 4 -> 11
- net +5V: track 88.5 -> 264.9 mm, vias 4 -> 6
- net DRV2_SCL: track 0.00 -> 142.8 mm, vias 0 -> 3
- net DRV2_SDA: track 0.00 -> 141.5 mm, vias 0 -> 2
- net DRV1_SCL: track 10.4 -> 51.5 mm
- net GND: track 85.5 -> 121.5 mm, vias 435 -> 529
- net DRV1_SDA: track 10.0 -> 45.1 mm, vias 0 -> 2
- net CS5: track 148.2 -> 150.4 mm
- net Net-(D2-A): track 1.55 -> 3.53 mm
- net Net-(U2-RSET): track 0.00 -> 0.88 mm
- net Green1: track 155.7 -> 156.5 mm
- net Net-(U1-RSET): track 1.74 -> 1.06 mm
- net Net-(U2-IICRST): track 2.48 -> 1.83 mm
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- added copper zone on In3.Cu, net GND
- added copper zone on In4.Cu, net GND
- removed copper zone on In2.Cu, net GND
Other:
- copper layers 4 -> 6
