File: Chord Board Controller.kicad_pcb (KiCad board)
At the start: 6 copper layers, 207 x 149.9 mm, 215 parts, among them J1 5 Pin Header 2.54mm, J4 HRO_TYPE-C-31-M-14, J8 Batt_1S, Q13 2N7002, SW1 RotaryEncoder_Switch, SW2 RotaryEncoder_Switch, SW3 RotaryEncoder_Switch, SW4 RotaryEncoder_Switch, SW5 RotaryEncoder_Switch, SW6 SW_SPST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

Commit message: aron review
Parts:
- moved H7 15.7 mm to (245.8, 55.1)
- moved H2 1.58 mm to (122.1, 121.5)
- moved H1 1.28 mm to (229.4, 121.5)
- moved H3 0.74 mm to (263.9, 148.6)
- moved H4 0.74 mm to (88.6, 148.6)
- moved H6 0.42 mm to (111.4, 55.5)
Routing:
- net +3.3V: track 246.9 -> 280.9 mm, vias 11 -> 12
- net GND: track 121.5 -> 125.3 mm, vias 529 -> 548
- net Red2: track 73.8 -> 76.1 mm
- net +VUSB: track 119.9 -> 118.5 mm
- net DRV1_SDA: track 45.1 -> 46.1 mm
